File: Micromouse2026PCB/Micromouse2026PCB.kicad_pcb (KiCad board)
At the start: 2 copper layers, 109.2 x 68.6 mm, 18 parts, among them J1 Power Terminal, J2 i2c OLED, J3 BNO085, SW1 PowerSW

Commit message: AAAAAAAAAAAAAAAAAA
Parts:
- moved A1 71.3 mm to (107.2, 24.0), turned to -90 degrees
- moved D1 69.6 mm to (108.0, 76.2)
- moved RS1 49.3 mm to (88.0, 28.6)
- moved J2 26.9 mm to (80.0, 61.0)
- moved J3 11.4 mm to (54.6, 48.3)
- moved R2 10.3 mm to (122.6, 85.1)
- moved J1 4.84 mm to (107.3, 81.9), turned to -90 degrees
- moved R1 4.26 mm to (122.6, 81.3)
- moved U1 3.81 mm to (35.6, 83.8)
- moved U5 3.81 mm to (48.3, 30.5)
Routing:
- net Net-(M1-OB): track 20.3 -> 189.2 mm
- net Net-(U2-XSHUT): track 60.1 -> 165.4 mm
- net Net-(MD1-IB): track 29.7 -> 129.9 mm, vias 0 -> 1
- net Net-(MD1-IA): track 34.5 -> 132.3 mm, vias 0 -> 1
- net Net-(A1-D0/RX): track 20.8 -> 100.3 mm
- net Net-(D1-K): track 103.4 -> 26.8 mm, vias 0 -> 1
- net Net-(U4-XSHUT): track 99.4 -> 168.9 mm, vias 1 -> 0
- net Net-(U1-XSHUT): track 42.0 -> 102.1 mm, vias 0 -> 1
- net Net-(A1-PadD4): track 88.8 -> 41.8 mm
- net /SCL: track 250.1 -> 295.3 mm, vias 0 -> 1
- net Net-(D1-A): track 70.5 -> 26.5 mm
- net Net-(U3-XSHUT): track 63.1 -> 106.1 mm
- net Net-(MD2-IA): track 67.1 -> 108.6 mm, vias 1 -> 0
- net +5V: track 346.7 -> 326.0 mm
- net Net-(A1-PadD8): track 76.0 -> 55.9 mm
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Other:
- outline, holes or cut-outs redrawn
- board text added: "Knuth"
- board text added: "Micromouse 3.0 Polyphemus - Bailey Cash - Ethan Joshua - Lucy"
