File: Micromouse2026PCB/Micromouse2026PCB.kicad_sch (KiCad schematic)
At the start: 0 parts

Commit message: started pcb work and custom symbols
Parts:
- added A1: Arduino_Micro_Socket, PCM_arduino-library:Arduino_Micro_Socket, symbol PCM_arduino-library:Arduino_Micro_Socket
- added J1: Power Terminal, Connector_PinHeader_2.54mm:PinHeader_1x06_P2.54mm_Vertical, symbol Connector:Screw_Terminal_01x02
- added MD1, MD2: (no value), Package_DIP:DIP-8_W7.62mm_Socket, symbol CustomSym:L9110H
- added U1, U2, U3, U4, U5: (no value), Connector_PinHeader_2.54mm:PinHeader_1x06_P2.54mm_Vertical, symbol CustomSym:VL53L0X_Breakout
- added U6: L7805, symbol Regulator_Linear:L7805
Connections:
- new net: A1.A0, U1.6 (XSHUT)
- new net: A1.A1, U2.6 (XSHUT)
- new net: A1.A2, U3.6 (XSHUT)
- new net: A1.A3, U4.6 (XSHUT)
- new net: A1.VIN, J1.1 (Pin_1), U6.1 (IN)
- new net: MD1.2 (VCC), MD1.3 (VCC), MD2.2 (VCC), MD2.3 (VCC), U6.3 (OUT)
- new net +3.3V: A1.3V3 (3.3V)
- new net +5V: A1.5V, U1.1 (VIN), U2.1 (VIN), U3.1 (VIN), U4.1 (VIN), U5.1 (VIN)
- new net GND: A1.GND1 (GND), A1.GND2 (GND), J1.2 (Pin_2), MD1.5 (GND), MD1.8 (GND), MD2.5 (GND), MD2.8 (GND), U1.2 (GND), U2.2 (GND), U3.2 (GND), U4.2 (GND), U5.2 (GND), U6.2 (GND)
- new net SCL: A1.D3 (D3/SCL), U1.3 (SCL), U2.3 (SCL), U3.3 (SCL), U4.3 (SCL), U5.3 (SCL)
- new net SDA: A1.D2 (D2/SDA), U1.4 (SDA), U2.4 (SDA), U3.4 (SDA), U4.4 (SDA), U5.4 (SDA)
- no-connect marks 0 -> 6

Commit message: worked on PCB
Parts:
- added J2: i2c OLED, Connector:FanPinHeader_1x04_P2.54mm_Vertical, symbol Connector:Conn_01x04_Pin
- added M1, M2: (no value), Connector_JST:JST_ZH_B6B-ZR_1x06_P1.50mm_Vertical, symbol CustomSym:GearMotor
- J1: footprint Connector_PinHeader_2.54mm:PinHeader_1x06_P2.54mm_Vertical -> TerminalBlock_Phoenix:TerminalBlock_Phoenix_MKDS-1,5-2-5.08_1x02_P5.08mm_Horizontal
- U6: footprint (none) -> Package_TO_SOT_THT:TO-220-3_Vertical
Connections:
- net +5V: now also J2.2 (Pin_2), M1.3 (VCC), M2.3 (VCC)
- net GND: now also J2.1 (Pin_1), M1.4 (GND), M2.4 (GND)
- net SCL: now also J2.3 (Pin_3)
- net SDA: now also J2.4 (Pin_4)
- net at MD1.6 (IA): now also M1.1 (MA)
- net at MD1.7 (IB): now also M1.2 (MB)
- net at MD2.6 (IA): now also M2.1 (MA)
- net at MD2.7 (IB): now also M2.2 (MB)

Commit message: New PCB work
Parts:
- added J3: BNO085, Connector_PinHeader_2.54mm:PinHeader_1x06_P2.54mm_Vertical, symbol Connector:Conn_01x06_Pin
- added SW1: RotaryEncoder_Switch, symbol Device:RotaryEncoder_Switch
- J2: footprint Connector:FanPinHeader_1x04_P2.54mm_Vertical -> Connector_PinHeader_2.54mm:PinHeader_1x04_P2.54mm_Vertical
Connections:
- net +5V: now also J3.1 (Pin_1)
- net GND: now also J3.3 (Pin_3), SW1.C
- net SCL: now also J3.4 (Pin_4)
- net SDA: now also J3.5 (Pin_5)
- net at A1.A4: now also M1.6 (OB)
- net at A1.A5: now also M2.6 (OB)
- net at A1.D0 (D0/RX): now also M2.5 (OA)
- net at A1.D1 (D1/TX): now also M1.5 (OA)
- net at A1.D10: now also MD2.7 (IB)
- net at A1.D5: now also MD1.6 (IA)
- net at A1.D6: now also MD1.7 (IB)
- net at A1.D9: now also MD2.6 (IA)
- net at M2.1 (MA): now also MD2.1 (OA); no longer MD2.6 (IA)
- net at M2.2 (MB): now also MD2.4 (OB); no longer MD2.7 (IB)
- net at MD1.1 (OA): now also M1.1 (MA)
- net at MD1.4 (OB): now also M1.2 (MB)
- no-connect marks 6 -> 8
Other:
- moved on the sheet: A1, M2

Commit message: finished schematic
Parts:
- SW1: footprint (none) -> Rotary_Encoder:RotaryEncoder_Alps_EC11E-Switch_Vertical_H20mm
Connections:
- net GND: now also SW1.S2
- net at A1.D4: now also SW1.S1
- net at A1.D7 (D7_INT4): now also SW1.A
- net at A1.D8: now also SW1.B
- no-connect marks 8 -> 18

Commit message: PCB work
Parts:
- J2: footprint Connector_PinHeader_2.54mm:PinHeader_1x04_P2.54mm_Vertical -> CustomFootprints:OLED_0.96_SSD1306_I2C
- J3: footprint Connector_PinHeader_2.54mm:PinHeader_1x06_P2.54mm_Vertical -> CustomFootprints:Adafruit_BNO085
Changed lines of the file:
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@@
 			)
 		)
-		(property "Footprint" "Connector_PinHeader_2.54mm:PinHeader_1x06_P2.54mm_Vertical"
+		(property "Footprint" "CustomFootprints:Adafruit_BNO085"
 			(at 101.6 48.26 0)
 			(hide yes)
@@
 			)
 		)
-		(property "Footprint" "Connector_PinHeader_2.54mm:PinHeader_1x04_P2.54mm_Vertical"
+		(property "Footprint" "CustomFootprints:OLED_0.96_SSD1306_I2C"
 			(at 101.6 69.85 0)
 			(hide yes)

Commit message: PCB working version
Parts:
- removed U6: L7805, Package_TO_SOT_THT:TO-220-3_Vertical, symbol Regulator_Linear:L7805
- added D1: 1N5822, Diode_THT:D_DO-201AD_P15.24mm_Horizontal, symbol Diode:1N5822
- added R1, R2: 10k, Resistor_THT:R_Axial_DIN0207_L6.3mm_D2.5mm_P10.16mm_Horizontal, symbol Device:R
- added SW1: PowerSW, Connector_PinHeader_2.54mm:PinHeader_1x03_P2.54mm_Vertical, symbol Connector_Generic:Conn_01x03
- J1: footprint TerminalBlock_Phoenix:TerminalBlock_Phoenix_MKDS-1,5-2-5.08_1x02_P5.08mm_Horizontal -> TerminalBlock_Phoenix:TerminalBlock_Phoenix_MPT-0,5-2-2.54_1x02_P2.54mm_Horizontal
- renumbered SW1 to RS1
Connections:
- net GND: now also R2.2
- net at A1.A4: no longer M1.6 (OB)
- net at A1.A5: now also R1.2, R2.1; no longer M2.6 (OB)
- net at A1.D11: now also M2.6 (OB)
- net at A1.D12: now also M1.6 (OB)
- net at A1.VIN: now also MD1.2 (VCC), MD1.3 (VCC), MD2.2 (VCC), MD2.3 (VCC), R1.1, SW1.1 (Pin_1); no longer J1.1 (Pin_1)
- new net: D1.1 (K), SW1.2 (Pin_2)
- new net: D1.2 (A), J1.1 (Pin_1)
Other:
- moved on the sheet: J1, RS1

Commit message: AAAAAAAAAAAAAAAAAA
Connections:
- net at A1.A4: now also U5.6 (XSHUT)
- no-connect marks 18 -> 16
Changed lines of the file:
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@@
-	)
-	(no_connect
-		(at 143.51 85.09)
 	)
 	(no_connect
@@
 	)
 	(no_connect
-		(at 82.55 81.28)
-	)
-	(no_connect
 		(at 194.31 90.17)
 	)
@@
 	(wire
 		(pts
+			(xy 143.51 85.09) (xy 82.55 85.09)
+		)
+		(stroke
+			(width 0)
+			(type default)
+		)
+	)
+	(wire
+		(pts
 			(xy 110.49 102.87) (xy 143.51 102.87)
 		)
@@
 		)
 		(stroke
+			(width 0)
+			(type default)
+		)
+	)
+	(wire
+		(pts
+			(xy 82.55 85.09) (xy 82.55 81.28)
+		)
+		(stroke
